File: RDpico_electronics/RDpico_PS/RD56m_PS_V1.kicad_sch (KiCad schematic)
At the start: 25 parts, among them J1 Barrel_Jack_Switch_Pin3Ring, M1 Motor_DC, Q1 NPN, Q2 NPN, SW1 SW_DPDT_x2, U1 Pin-Connector, U2 Pin-Connector, U3 Pin-Connector, U4 Pin-Connector, U5 Pin-Connector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

Commit message: BOM completed
Parts:
- R2: value 47 -> 100
- R3: value 120 -> 270
- RV1: value 470 -> 1k
Changed lines of the file:
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@@
       (effects (font (size 1.27 1.27)))
     )
-    (property "Value" "470" (at 134.62 134.62 0)
+    (property "Value" "1k" (at 134.62 134.62 0)
       (effects (font (size 1.27 1.27)))
     )
@@
       (effects (font (size 1.27 1.27)) (justify left))
     )
-    (property "Value" "120" (at 132.588 114.173 0)
+    (property "Value" "270" (at 132.588 114.173 0)
       (effects (font (size 1.27 1.27)) (justify left))
     )
@@
       (effects (font (size 1.27 1.27)) (justify left))
     )
-    (property "Value" "47" (at 132.588 125.603 0)
-      (effects (font (size 1.27 1.27)) (justify left))
-    )
+    (property "Value" "100" (at 132.588 125.603 0)
+      (effects (font (size 1.27 1.27)) (justify left))
+    )
