File: RDpico_electronics/RDpico_display/LED1.kicad_sch (KiCad schematic)
At the start: 77 parts, among them Q1 IRLML6401, Q10 BS250, Q12 BS250, Q14 BS250, Q2 BS250, Q4 BS250, Q6 BS250, Q8 BS250

Commit message: update production files
Parts:
- Q1: LCSC (none) -> C2835446
Changed lines of the file:
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@@
       (effects (font (size 1.27 1.27)) (justify left) hide)
+    )
+    (property "LCSC" "C2835446" (at 119.38 34.29 0)
+      (effects (font (size 1.27 1.27)) hide)
     )
     (pin "1")
@@
       (effects (font (size 1.27 1.27)) (justify left) hide)
     )
+    (property "LCSC" "C2835446" (at 119.38 109.22 0)
+      (effects (font (size 1.27 1.27)) hide)
+    )
     (pin "1")
     (pin "2")
@@
     (property "Datasheet" "https://www.infineon.com/dgdl/irlml6401pbf.pdf?fileId=5546d462533600a401535668b96d2634" (at 220.98 34.29 0)
       (effects (font (size 1.27 1.27)) (justify left) hide)
+    )
+    (property "LCSC" "C2835446" (at 220.98 34.29 0)
+      (effects (font (size 1.27 1.27)) hide)
     )
     (pin "1")
@@
       (effects (font (size 1.27 1.27)) (justify left) hide)
     )
+    (property "LCSC" "C2835446" (at 68.58 34.29 0)
+      (effects (font (size 1.27 1.27)) hide)
+    )
     (pin "1")
     (pin "2")
@@
       (effects (font (size 1.27 1.27)) (justify left) hide)
     )
+    (property "LCSC" "C2835446" (at 170.18 34.29 0)
+      (effects (font (size 1.27 1.27)) hide)
+    )
     (pin "1")
     (pin "2")
@@
       (effects (font (size 1.27 1.27)) (justify left) hide)
     )
+    (property "LCSC" "C2835446" (at 170.18 109.22 0)
+      (effects (font (size 1.27 1.27)) hide)
+    )
     (pin "1")
     (pin "2")
@@
       (effects (font (size 1.27 1.27)) (justify left) hide)
     )
-    (pin "1")
+    (property "LCSC" "C2835446" (at 68.58 109.22 0)
+      (effects (font (size 1.27 1.27)) hide)
+    )
+    (pin "1")
